Commit message: Add AMCL localization files for Where Am I project

File: my_robot/urdf/my_robot.xacro (robot description, xacro)
@@ -1,149 +1,175 @@
-<?xml version="1.0"?>
+<?xml version='1.0'?>
 <robot name="my_robot" xmlns:xacro="http://www.ros.org/wiki/xacro">
-  <material name="yellow">
-    <color rgba="1 1 0 1"/>
-  </material>
-  <material name="black">
-    <color rgba="0 0 0 1"/>
-  </material>
-  <material name="white">
-    <color rgba="1 1 1 1"/>
-  </material>
-  <link name="base_link">
-    <visual>
-      <origin xyz="0 0 0.05" rpy="0 0 0.785"/>
-      <geometry>
-        <box size="0.42 0.42 0.12"/>
-      </geometry>
-      <material name="yellow"/>
-    </visual>
-    <collision>
-      <origin xyz="0 0 0.05" rpy="0 0 0.785"/>
-      <geometry>
-        <box size="0.42 0.42 0.12"/>
-      </geometry>
-    </collision>
-    <inertial>
-      <origin xyz="0 0 0.05"/>
-      <mass value="5.0"/>
-      <inertia ixx="0.1" ixy="0.0" ixz="0.0" iyy="0.1" iyz="0.0" izz="0.1"/>
-    </inertial>
-  </link>
-  <link name="left_wheel">
-    <visual>
-      <origin xyz="0 0 0" rpy="1.5707 0 0"/>
-      <geometry>
-        <cylinder radius="0.08" length="0.05"/>
-      </geometry>
-      <material name="black"/>
-    </visual>
-    <collision>
-      <origin xyz="0 0 0" rpy="1.5707 0 0"/>
-      <geometry>
-        <cylinder radius="0.08" length="0.05"/>
-      </geometry>
-    </collision>
-    <inertial>
-      <mass value="1.0"/>
-      <inertia ixx="0.01" ixy="0.0" ixz="0.0" iyy="0.01" iyz="0.0" izz="0.01"/>
-    </inertial>
-  </link>
-  <link name="right_wheel">
-    <visual>
-      <origin xyz="0 0 0" rpy="1.5707 0 0"/>
-      <geometry>
-        <cylinder radius="0.08" length="0.05"/>
-      </geometry>
-      <material name="black"/>
-    </visual>
-    <collision>
-      <origin xyz="0 0 0" rpy="1.5707 0 0"/>
-      <geometry>
-        <cylinder radius="0.08" length="0.05"/>
-      </geometry>
-    </collision>
-    <inertial>
-      <mass value="1.0"/>
-      <inertia ixx="0.01" ixy="0.0" ixz="0.0" iyy="0.01" iyz="0.0" izz="0.01"/>
-    </inertial>
-  </link>
-  <joint name="left_wheel_joint" type="continuous">
-    <origin xyz="0 0.18 0.02" rpy="0 0 0"/>
-    <parent link="base_link"/>
+<xacro:include filename="$(find my_robot)/urdf/my_robot.gazebo" />
+                                                  <link name="robot_footprint"></link>
+                                                  <joint name="robot_footprint_joint" type="fixed">
+                                                    <origin xyz="0 0 0" rpy="0 0 0" />
+                                                    <parent link="robot_footprint"/>
+                                                    <child link="chassis" />
+                                                  </joint>
+                                                  <link name='chassis'>
+                                                    <inertial>
+                                                      <mass value="15.0"/>
+                                                      <origin xyz="0.0 0 0" rpy=" 0 0 0"/>
+                                                      <inertia
+                                                          ixx="0.1" ixy="0" ixz="0"
+                                                          iyy="0.1" iyz="0"
+                                                          izz="0.1"
+                                                      />
+                                                    </inertial>
+                                                    <collision name='collision'>
+                                                      <origin xyz="0 0 0" rpy=" 0 0 0"/>
+                                                      <geometry>
+                                                        <box size=".8 .4 .2"/>
+                                                      </geometry>
+                                                    </collision>
+                                                    <visual name='chassis_visual'>
+                                                      <origin xyz="0 0 0" rpy=" 0 0 0"/>
+                                                      <geometry>
+                                                        <box size=".8 .4 .2"/>
+                                                      </geometry>
+                                                      <material name="blue">
+    								<color rgba="0 0 1 1"/>
+ 							 </material>
+                                                    </visual>
+                                                    <collision name='back_caster_collision'>
+                                                      <origin xyz="-0.15 0 -0.05" rpy=" 0 0 0"/>
+                                                      <geometry>
+                                                        <sphere radius="0.0499"/>
+                                                      </geometry>
+                                                    </collision>
+                                                    <visual name='back_caster_visual'>
+                                                      <origin xyz="-0.15 0 -0.05" rpy=" 0 0 0"/>
+                                                      <geometry>
+                                                        <sphere radius="0.05"/>
+                                                      </geometry>
+                                                    </visual>
+                                                    <collision name='front_caster_collision'>
+                                                      <origin xyz="0.15 0 -0.05" rpy=" 0 0 0"/>
+                                                      <geometry>
+                                                        <sphere radius="0.0499"/>
+                                                      </geometry>
+                                                    </collision>
+                                                    <visual name='front_caster_visual'>
+                                                      <origin xyz="0.15 0 -0.05" rpy=" 0 0 0"/>
+                                                      <geometry>
+                                                        <sphere radius="0.05"/>
+                                                      </geometry>
+                                                    </visual>
+                                                  </link>
+<link name="left_wheel">
+  <inertial>
+    <mass value="5"/>
+    <origin xyz="0 0 0" rpy="0 1.5707 1.5707"/>
+    <inertia
+      ixx="0.1" ixy="0" ixz="0"
+      iyy="0.1" iyz="0"
+      izz="0.1"/>
+  </inertial>
+  <collision name="left_wheel_collision">
+    <origin xyz="0 0 0" rpy="0 1.5707 1.5707"/>
+    <geometry>
+      <cylinder radius="0.05" length="0.05"/>
+    </geometry>
+  </collision>
+  <visual name="left_wheel_visual">
+    <origin xyz="0 0 0" rpy="0 1.5707 1.5707"/>
+    <geometry>
+      <cylinder radius="0.05" length="0.05"/>
+    </geometry>
+  </visual>
+</link>
+<link name="right_wheel">
+  <inertial>
+    <mass value="5"/>
+    <origin xyz="0 0 0" rpy="0 1.5707 1.5707"/>
+    <inertia
+      ixx="0.1" ixy="0" ixz="0"
+      iyy="0.1" iyz="0"
+      izz="0.1"/>
+  </inertial>
+  <collision name="right_wheel_collision">
+    <origin xyz="0 0 0" rpy="0 1.5707 1.5707"/>
+    <geometry>
+      <cylinder radius="0.05" length="0.05"/>
+    </geometry>
+  </collision>
+  <visual name="right_wheel_visual">
+    <origin xyz="0 0 0" rpy="0 1.5707 1.5707"/>
+    <geometry>
+      <cylinder radius="0.05" length="0.05"/>
+    </geometry>
+  </visual>
+</link>
+<link name="camera">
+  <inertial>
+    <mass value="0.1"/>
+    <origin xyz="0 0 0" rpy="0 0 0"/>
+    <inertia
+      ixx="1e-6" ixy="0" ixz="0"
+      iyy="1e-6" iyz="0"
+      izz="1e-6"/>
+  </inertial>
+  <collision name="camera_collision">
+    <origin xyz="0 0 0" rpy="0 0 0"/>
+    <geometry>
+      <box size="0.05 0.05 0.05"/>
+    </geometry>
+  </collision>
+  <visual name="camera_visual">
+    <origin xyz="0 0 0" rpy="0 0 0"/>
+    <geometry>
+      <box size="0.05 0.05 0.05"/>
+    </geometry>
+  </visual>
+</link>
+<joint name="camera_joint" type="fixed">
+  <origin xyz="0.2 0 0.1" rpy="0 0 0"/>
+  <parent link="chassis"/>
+  <child link="camera"/>
+</joint>
+<link name="hokuyo">
+  <inertial>
+    <mass value="1e-5"/>
+    <origin xyz="0 0 0" rpy="0 0 0"/>
+    <inertia
+      ixx="1e-6" ixy="0" ixz="0"
+      iyy="1e-6" iyz="0"
+      izz="1e-6"/>
+  </inertial>
+  <collision name="hokuyo_collision">
+    <origin xyz="0 0 0" rpy="0 0 0"/>
+    <geometry>
+      <box size="0.1 0.1 0.1"/>
+    </geometry>
+  </collision>
+  <visual name="hokuyo_visual">
+    <origin xyz="0 0 0" rpy="0 0 0"/>
+    <geometry>
+      <mesh filename="package://my_robot/meshes/hokuyo.dae"/>
+    </geometry>
+  </visual>
+</link>
+<joint name="hokuyo_joint" type="fixed">
+  <origin xyz="0.15 0 0.1" rpy="0 0 0"/>
+  <parent link="chassis"/>
+  <child link="hokuyo"/>
+  <axis xyz="0 1 0"/>
+</joint>
+ <joint type="continuous" name="left_wheel_hinge">
+    <origin xyz="0 0.15 -0.1" rpy="0 0 0"/>
     <child link="left_wheel"/>
+    <parent link="chassis"/>
     <axis xyz="0 1 0"/>
+    <limit effort="10000" velocity="1000"/>
+    <dynamics damping="1.0" friction="1.0"/>
   </joint>
-  <joint name="right_wheel_joint" type="continuous">
-    <origin xyz="0 -0.18 0.02" rpy="0 0 0"/>
-    <parent link="base_link"/>
+ <joint type="continuous" name="right_wheel_hinge">
+    <origin xyz="0 -0.15 -0.1" rpy="0 0 0"/>
     <child link="right_wheel"/>
+    <parent link="chassis"/>
     <axis xyz="0 1 0"/>
+    <limit effort="10000" velocity="1000"/>
+    <dynamics damping="1.0" friction="1.0"/>
   </joint>
-  <link name="caster">
-    <visual>
-      <geometry>
-        <sphere radius="0.03"/>
-      </geometry>
-      <material name="black"/>
-    </visual>
-    <collision>
-      <geometry>
-        <sphere radius="0.03"/>
-      </geometry>
-    </collision>
-    <inertial>
-      <mass value="0.3"/>
-      <inertia ixx="0.001" ixy="0.0" ixz="0.0" iyy="0.001" iyz="0.0" izz="0.001"/>
-    </inertial>
-  </link>
-  <joint name="caster_joint" type="fixed">
-    <origin xyz="-0.16 0 -0.01" rpy="0 0 0"/>
-    <parent link="base_link"/>
-    <child link="caster"/>
-  </joint>
-  <link name="camera_link">
-    <visual>
-      <geometry>
-        <box size="0.05 0.05 0.05"/>
-      </geometry>
-      <material name="white"/>
-    </visual>
-    <collision>
-      <geometry>
-        <box size="0.05 0.05 0.05"/>
-      </geometry>
-    </collision>
-    <inertial>
-      <mass value="0.2"/>
-      <inertia ixx="0.001" ixy="0.0" ixz="0.0" iyy="0.001" iyz="0.0" izz="0.001"/>
-    </inertial>
-  </link>
-  <joint name="camera_joint" type="fixed">
-    <origin xyz="0.16 0 0.14" rpy="0 0 0"/>
-    <parent link="base_link"/>
-    <child link="camera_link"/>
-  </joint>
-  <link name="laser_link">
-    <visual>
-      <geometry>
-        <cylinder radius="0.03" length="0.05"/>
-      </geometry>
-      <material name="white"/>
-    </visual>
-    <collision>
-      <geometry>
-        <cylinder radius="0.03" length="0.05"/>
-      </geometry>
-    </collision>
-    <inertial>
-      <mass value="0.2"/>
-      <inertia ixx="0.001" ixy="0.0" ixz="0.0" iyy="0.001" iyz="0.0" izz="0.001"/>
-    </inertial>
-  </link>
-  <joint name="laser_joint" type="fixed">
-    <origin xyz="0.10 0 0.14" rpy="0 0 0"/>
-    <parent link="base_link"/>
-    <child link="laser_link"/>
-  </joint>
-  <xacro:include filename="$(find my_robot)/urdf/my_robot.gazebo"/>
 </robot>

Commit message: Backup robotics workspace

File: my_robot/urdf/my_robot.xacro (robot description, xacro)
@@ -4,5 +4,5 @@
                                                   <link name="robot_footprint"></link>
                                                   <joint name="robot_footprint_joint" type="fixed">
-                                                    <origin xyz="0 0 0" rpy="0 0 0" />
+                                                    <origin xyz="0 0 0.1" rpy="0 0 0" />
                                                     <parent link="robot_footprint"/>
                                                     <child link="chassis" />
@@ -34,5 +34,5 @@
                                                     </visual>
                                                     <collision name='back_caster_collision'>
-                                                      <origin xyz="-0.15 0 -0.05" rpy=" 0 0 0"/>
+                                                      <origin xyz="-0.15 0 -0.1" rpy=" 0 0 0"/>
                                                       <geometry>
                                                         <sphere radius="0.0499"/>
@@ -40,5 +40,5 @@
                                                     </collision>
                                                     <visual name='back_caster_visual'>
-                                                      <origin xyz="-0.15 0 -0.05" rpy=" 0 0 0"/>
+                                                      <origin xyz="-0.15 0 -0.1" rpy=" 0 0 0"/>
                                                       <geometry>
                                                         <sphere radius="0.05"/>
@@ -46,5 +46,5 @@
                                                     </visual>
                                                     <collision name='front_caster_collision'>
-                                                      <origin xyz="0.15 0 -0.05" rpy=" 0 0 0"/>
+                                                      <origin xyz="0.15 0 -0.1" rpy=" 0 0 0"/>
                                                       <geometry>
                                                         <sphere radius="0.0499"/>
@@ -52,5 +52,5 @@
                                                     </collision>
                                                     <visual name='front_caster_visual'>
-                                                      <origin xyz="0.15 0 -0.05" rpy=" 0 0 0"/>
+                                                      <origin xyz="0.15 0 -0.1" rpy=" 0 0 0"/>
                                                       <geometry>
                                                         <sphere radius="0.05"/>
